File: OpenPowerDistributor/3.3V internal supply.kicad_sch (KiCad schematic)
At the start: 8 parts, among them U6 AP63200WU

Commit message: Added LEDs
Parts:
- renumbered C20 to C1, C21 to C2, C22 to C3, D4 to D3, L2 to L1, R18 to R1, R15 to R2, U6 to U1
Changed lines of the file:
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@@
   (symbol (lib_id "Regulator_Switching:AP63200WU") (at 100.33 83.82 0) (unit 1)
     (in_bom yes) (on_board yes) (dnp no) (fields_autoplaced)
-    (property "Reference" "U6" (at 100.33 73.025 0)
+    (property "Reference" "U1" (at 100.33 73.025 0)
       (effects (font (size 1.27 1.27)))
     )
@@
   (symbol (lib_id "power:GND") (at 196.85 92.71 0) (unit 1)
     (in_bom yes) (on_board yes) (dnp no) (fields_autoplaced)
-    (property "Reference" "#PWR049" (at 196.85 99.06 0)
+    (property "Reference" "#PWR08" (at 196.85 99.06 0)
       (effects (font (size 1.27 1.27)) hide)
     )
@@
   (symbol (lib_id "Diode:SMF48A") (at 196.85 87.63 270) (unit 1)
     (in_bom yes) (on_board yes) (dnp no) (fields_autoplaced)
-    (property "Reference" "D4" (at 199.39 86.3599 90)
+    (property "Reference" "D3" (at 199.39 86.3599 90)
       (effects (font (size 1.27 1.27)) (justify left))
     )
@@
   (symbol (lib_id "power:GND") (at 100.33 91.44 0) (unit 1)
     (in_bom yes) (on_board yes) (dnp no) (fields_autoplaced)
-    (property "Reference" "#PWR058" (at 100.33 97.79 0)
+    (property "Reference" "#PWR04" (at 100.33 97.79 0)
       (effects (font (size 1.27 1.27)) hide)
     )
@@
   (symbol (lib_id "Device:L_Ferrite") (at 140.97 83.82 90) (unit 1)
     (in_bom yes) (on_board yes) (dnp no) (fields_autoplaced)
-    (property "Reference" "L2" (at 140.97 76.835 90)
+    (property "Reference" "L1" (at 140.97 76.835 90)
       (effects (font (size 1.27 1.27)))
     )
@@
   (symbol (lib_id "Device:C_Small") (at 123.19 83.82 270) (mirror x) (unit 1)
     (in_bom yes) (on_board yes) (dnp no)
-    (property "Reference" "C20" (at 124.46 82.55 90)
+    (property "Reference" "C1" (at 124.46 82.55 90)
       (effects (font (size 1.27 1.27)) (justify left))
     )
@@
   (symbol (lib_id "Device:R_Small") (at 162.56 95.25 0) (unit 1)
     (in_bom yes) (on_board yes) (dnp no) (fields_autoplaced)
-    (property "Reference" "R15" (at 165.1 93.9799 0)
+    (property "Reference" "R2" (at 165.1 93.9799 0)
       (effects (font (size 1.27 1.27)) (justify left))
     )
@@
   (symbol (lib_id "Device:C_Polarized_Small") (at 180.34 86.36 0) (unit 1)
     (in_bom yes) (on_board yes) (dnp no) (fields_autoplaced)
-    (property "Reference" "C22" (at 182.88 84.5438 0)
+    (property "Reference" "C3" (at 182.88 84.5438 0)
       (effects (font (size 1.27 1.27)) (justify left))
     )
@@
   (symbol (lib_id "power:GND") (at 162.56 99.06 0) (unit 1)
     (in_bom yes) (on_board yes) (dnp no) (fields_autoplaced)
-    (property "Reference" "#PWR049" (at 162.56 105.41 0)
+    (property "Reference" "#PWR06" (at 162.56 105.41 0)
       (effects (font (size 1.27 1.27)) hide)
     )
@@
   (symbol (lib_id "Device:R_Small") (at 162.56 87.63 0) (unit 1)
     (in_bom yes) (on_board yes) (dnp no) (fields_autoplaced)
-    (property "Reference" "R18" (at 165.1 86.3599 0)
+    (property "Reference" "R1" (at 165.1 86.3599 0)
       (effects (font (size 1.27 1.27)) (justify left))
     )
@@
   (symbol (lib_id "Device:C_Small") (at 149.86 87.63 0) (unit 1)
     (in_bom yes) (on_board yes) (dnp no) (fields_autoplaced)
-    (property "Reference" "C21" (at 152.4 86.3662 0)
+    (property "Reference" "C2" (at 152.4 86.3662 0)
       (effects (font (size 1.27 1.27)) (justify left))
     )
@@
   (symbol (lib_id "power:GND") (at 180.34 88.9 0) (unit 1)
     (in_bom yes) (on_board yes) (dnp no) (fields_autoplaced)
-    (property "Reference" "#PWR059" (at 180.34 95.25 0)
-      (effects (font (size 1.27 1.27)) hide)
-    )
+    (property "Reference" "#PWR05" (at 180.34 95.25 0)
+      (effects (font (size 1.27 1.27)) hide)
+    )

Commit message: Start to make layout
Parts:
- renumbered C1 to C6, C2 to C7, C3 to C8, L1 to L2, R1 to R3, R2 to R4, U1 to U2
Changed lines of the file:
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@@
   (symbol (lib_id "Regulator_Switching:AP63200WU") (at 100.33 83.82 0) (unit 1)
     (in_bom yes) (on_board yes) (dnp no) (fields_autoplaced)
-    (property "Reference" "U1" (at 100.33 73.025 0)
+    (property "Reference" "U2" (at 100.33 73.025 0)
       (effects (font (size 1.27 1.27)))
     )
@@
       (project "OpenPowerDistribution"
         (path "/df87b081-37a2-452c-8581-7eff2c408a17/a4c605b7-0bb6-4343-96e8-12ac057a7ce8"
-          (reference "U1") (unit 1)
+          (reference "U2") (unit 1)
         )
       )
@@
   (symbol (lib_id "power:GND") (at 196.85 92.71 0) (unit 1)
     (in_bom yes) (on_board yes) (dnp no) (fields_autoplaced)
-    (property "Reference" "#PWR08" (at 196.85 99.06 0)
+    (property "Reference" "#PWR016" (at 196.85 99.06 0)
       (effects (font (size 1.27 1.27)) hide)
     )
@@
       (project "OpenPowerDistribution"
         (path "/df87b081-37a2-452c-8581-7eff2c408a17/a4c605b7-0bb6-4343-96e8-12ac057a7ce8"
-          (reference "#PWR08") (unit 1)
+          (reference "#PWR016") (unit 1)
         )
       )
@@
   (symbol (lib_id "power:GND") (at 100.33 91.44 0) (unit 1)
     (in_bom yes) (on_board yes) (dnp no) (fields_autoplaced)
-    (property "Reference" "#PWR04" (at 100.33 97.79 0)
+    (property "Reference" "#PWR012" (at 100.33 97.79 0)
       (effects (font (size 1.27 1.27)) hide)
     )
@@
       (project "OpenPowerDistribution"
         (path "/df87b081-37a2-452c-8581-7eff2c408a17/a4c605b7-0bb6-4343-96e8-12ac057a7ce8"
-          (reference "#PWR04") (unit 1)
+          (reference "#PWR012") (unit 1)
         )
       )
@@
   (symbol (lib_id "Device:L_Ferrite") (at 140.97 83.82 90) (unit 1)
     (in_bom yes) (on_board yes) (dnp no) (fields_autoplaced)
-    (property "Reference" "L1" (at 140.97 76.835 90)
+    (property "Reference" "L2" (at 140.97 76.835 90)
       (effects (font (size 1.27 1.27)))
     )
@@
       (project "OpenPowerDistribution"
         (path "/df87b081-37a2-452c-8581-7eff2c408a17/a4c605b7-0bb6-4343-96e8-12ac057a7ce8"
-          (reference "L1") (unit 1)
+          (reference "L2") (unit 1)
         )
       )
@@
   (symbol (lib_id "Device:C_Small") (at 123.19 83.82 270) (mirror x) (unit 1)
     (in_bom yes) (on_board yes) (dnp no)
-    (property "Reference" "C1" (at 124.46 82.55 90)
+    (property "Reference" "C6" (at 124.46 82.55 90)
       (effects (font (size 1.27 1.27)) (justify left))
     )
@@
       (project "OpenPowerDistribution"
         (path "/df87b081-37a2-452c-8581-7eff2c408a17/a4c605b7-0bb6-4343-96e8-12ac057a7ce8"
-          (reference "C1") (unit 1)
+          (reference "C6") (unit 1)
         )
       )
@@
   (symbol (lib_id "power:+12V") (at 81.28 81.28 0) (unit 1)
     (in_bom yes) (on_board yes) (dnp no) (fields_autoplaced)
-    (property "Reference" "#PWR09" (at 81.28 85.09 0)
+    (property "Reference" "#PWR011" (at 81.28 85.09 0)
       (effects (font (size 1.27 1.27)) hide)
     )
@@
       (project "OpenPowerDistribution"
         (path "/df87b081-37a2-452c-8581-7eff2c408a17/a4c605b7-0bb6-4343-96e8-12ac057a7ce8"
-          (reference "#PWR09") (unit 1)
+          (reference "#PWR011") (unit 1)
         )
       )
@@
   (symbol (lib_id "Device:R_Small") (at 162.56 95.25 0) (unit 1)
     (in_bom yes) (on_board yes) (dnp no) (fields_autoplaced)
-    (property "Reference" "R2" (at 165.1 93.9799 0)
+    (property "Reference" "R4" (at 165.1 93.9799 0)
       (effects (font (size 1.27 1.27)) (justify left))
     )
@@
       (project "OpenPowerDistribution"
         (path "/df87b081-37a2-452c-8581-7eff2c408a17/a4c605b7-0bb6-4343-96e8-12ac057a7ce8"
-          (reference "R2") (unit 1)
+          (reference "R4") (unit 1)
         )
       )
@@
   (symbol (lib_id "Device:C_Polarized_Small") (at 180.34 86.36 0) (unit 1)
     (in_bom yes) (on_board yes) (dnp no) (fields_autoplaced)
-    (property "Reference" "C3" (at 182.88 84.5438 0)
+    (property "Reference" "C8" (at 182.88 84.5438 0)
       (effects (font (size 1.27 1.27)) (justify left))
     )
@@
       (project "OpenPowerDistribution"
         (path "/df87b081-37a2-452c-8581-7eff2c408a17/a4c605b7-0bb6-4343-96e8-12ac057a7ce8"
-          (reference "C3") (unit 1)
+          (reference "C8") (unit 1)
         )
       )
@@
   (symbol (lib_id "power:GND") (at 162.56 99.06 0) (unit 1)
     (in_bom yes) (on_board yes) (dnp no) (fields_autoplaced)
-    (property "Reference" "#PWR06" (at 162.56 105.41 0)
+    (property "Reference" "#PWR013" (at 162.56 105.41 0)
       (effects (font (size 1.27 1.27)) hide)
     )
@@
       (project "OpenPowerDistribution"
         (path "/df87b081-37a2-452c-8581-7eff2c408a17/a4c605b7-0bb6-4343-96e8-12ac057a7ce8"
-          (reference "#PWR06") (unit 1)
+          (reference "#PWR013") (unit 1)
         )
       )
@@
   (symbol (lib_id "Device:R_Small") (at 162.56 87.63 0) (unit 1)
     (in_bom yes) (on_board yes) (dnp no) (fields_autoplaced)
-    (property "Reference" "R1" (at 165.1 86.3599 0)
+    (property "Reference" "R3" (at 165.1 86.3599 0)
       (effects (font (size 1.27 1.27)) (justify left))
     )
@@
       (project "OpenPowerDistribution"
         (path "/df87b081-37a2-452c-8581-7eff2c408a17/a4c605b7-0bb6-4343-96e8-12ac057a7ce8"
-          (reference "R1") (unit 1)
+          (reference "R3") (unit 1)
         )
       )
@@
   (symbol (lib_id "power:+3.3V") (at 180.34 81.28 0) (unit 1)
     (in_bom yes) (on_board yes) (dnp no) (fields_autoplaced)
-    (property "Reference" "#PWR07" (at 180.34 85.09 0)
+    (property "Reference" "#PWR014" (at 180.34 85.09 0)
       (effects (font (size 1.27 1.27)) hide)
     )
@@
       (project "OpenPowerDistribution"
         (path "/df87b081-37a2-452c-8581-7eff2c408a17/a4c605b7-0bb6-4343-96e8-12ac057a7ce8"
-          (reference "#PWR07") (unit 1)
+          (reference "#PWR014") (unit 1)
         )
       )
@@
   (symbol (lib_id "Device:C_Small") (at 149.86 87.63 0) (unit 1)
     (in_bom yes) (on_board yes) (dnp no) (fields_autoplaced)
-    (property "Reference" "C2" (at 152.4 86.3662 0)
+    (property "Reference" "C7" (at 152.4 86.3662 0)
       (effects (font (size 1.27 1.27)) (justify left))
     )
@@
       (project "OpenPowerDistribution"
         (path "/df87b081-37a2-452c-8581-7eff2c408a17/a4c605b7-0bb6-4343-96e8-12ac057a7ce8"
-          (reference "C2") (unit 1)
+          (reference "C7") (unit 1)
         )
       )
@@
   (symbol (lib_id "power:GND") (at 180.34 88.9 0) (unit 1)
     (in_bom yes) (on_board yes) (dnp no) (fields_autoplaced)
-    (property "Reference" "#PWR05" (at 180.34 95.25 0)
+    (property "Reference" "#PWR015" (at 180.34 95.25 0)
       (effects (font (size 1.27 1.27)) hide)
     )
@@
       (project "OpenPowerDistribution"
         (path "/df87b081-37a2-452c-8581-7eff2c408a17/a4c605b7-0bb6-4343-96e8-12ac057a7ce8"
-          (reference "#PWR05") (unit 1)
-        )
-      )
+          (reference "#PWR015") (unit 1)
+        )
+      )
