File: OpenPowerDistributor/5V buck converter.kicad_sch (KiCad schematic)
At the start: 8 parts, among them U17 TPS565208DDA

Commit message: More work on schematic wiring
Parts:
- renumbered C9 to C53
Changed lines of the file:
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@@
   (symbol (lib_id "Device:C_Small") (at 125.73 74.93 0) (unit 1)
     (in_bom yes) (on_board yes) (dnp no) (fields_autoplaced)
-    (property "Reference" "C9" (at 128.27 73.6663 0)
+    (property "Reference" "C53" (at 128.27 73.6663 0)
       (effects (font (size 1.27 1.27)) (justify left))
     )
@@
     (instances
       (project "OpenPowerDistribution"
-        (path "/df87b081-37a2-452c-8581-7eff2c408a17/b96d46bc-8ba1-4cbe-b99e-e39dc05b303c"
-          (reference "C9") (unit 1)
-        )
-        (path "/df87b081-37a2-452c-8581-7eff2c408a17/e4deee11-55f7-4f18-af99-bea885b0cfea"
-          (reference "C17") (unit 1)
-        )
-        (path "/df87b081-37a2-452c-8581-7eff2c408a17/85719244-66a7-40c3-82ed-28faeb6fb371"
-          (reference "C22") (unit 1)
-        )
-        (path "/df87b081-37a2-452c-8581-7eff2c408a17/74fd09d3-df1f-43b2-92e6-36c41e96448f"
-          (reference "C27") (unit 1)
-        )
-        (path "/df87b081-37a2-452c-8581-7eff2c408a17/e5191bda-9cfb-4a55-9ca3-cd9bac3e48c3"
-          (reference "C42") (unit 1)
-        )
-        (path "/df87b081-37a2-452c-8581-7eff2c408a17/c66097e8-d629-4b84-bed3-ecef8eda3008"
-          (reference "C37") (unit 1)
-        )
-        (path "/df87b081-37a2-452c-8581-7eff2c408a17/f02926a4-ecb0-4085-b2d0-fb1538d188c5"
-          (reference "C32") (unit 1)
-        )
-        (path "/df87b081-37a2-452c-8581-7eff2c408a17/3d9b216d-734e-4ffd-941d-a104869460a4"
-          (reference "C52") (unit 1)
-        )
-        (path "/df87b081-37a2-452c-8581-7eff2c408a17/f529eff0-84d8-4678-a1b3-b1f91f6d1c09"
-          (reference "C47") (unit 1)
-        )
         (path "/df87b081-37a2-452c-8581-7eff2c408a17/e80d9cb1-99ed-4151-affe-23d60cb9d8e2"
           (reference "C53") (unit 1)

Commit message: Start to make layout
Parts:
- renumbered C56 to C5
Changed lines of the file:
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@@
         )
         (path "/df87b081-37a2-452c-8581-7eff2c408a17/c5ef4c26-c64f-4464-8506-0cba199ca76f"
-          (reference "C54") (unit 1)
+          (reference "C3") (unit 1)
         )
       )
@@
         )
         (path "/df87b081-37a2-452c-8581-7eff2c408a17/c5ef4c26-c64f-4464-8506-0cba199ca76f"
-          (reference "L3") (unit 1)
+          (reference "L1") (unit 1)
         )
       )
@@
         )
         (path "/df87b081-37a2-452c-8581-7eff2c408a17/c5ef4c26-c64f-4464-8506-0cba199ca76f"
-          (reference "R167") (unit 1)
+          (reference "R1") (unit 1)
         )
       )
@@
         )
         (path "/df87b081-37a2-452c-8581-7eff2c408a17/c5ef4c26-c64f-4464-8506-0cba199ca76f"
-          (reference "#PWR0159") (unit 1)
+          (reference "#PWR010") (unit 1)
         )
       )
@@
         )
         (path "/df87b081-37a2-452c-8581-7eff2c408a17/c5ef4c26-c64f-4464-8506-0cba199ca76f"
-          (reference "#PWR0154") (unit 1)
+          (reference "#PWR05") (unit 1)
         )
       )
@@
         )
         (path "/df87b081-37a2-452c-8581-7eff2c408a17/c5ef4c26-c64f-4464-8506-0cba199ca76f"
-          (reference "#PWR0156") (unit 1)
+          (reference "#PWR07") (unit 1)
         )
       )
@@
         )
         (path "/df87b081-37a2-452c-8581-7eff2c408a17/c5ef4c26-c64f-4464-8506-0cba199ca76f"
-          (reference "R168") (unit 1)
+          (reference "R2") (unit 1)
         )
       )
@@
   (symbol (lib_id "Device:C_Small") (at 166.37 80.01 0) (unit 1)
     (in_bom yes) (on_board yes) (dnp no)
-    (property "Reference" "C56" (at 163.83 78.7463 0)
+    (property "Reference" "C5" (at 163.83 78.7463 0)
       (effects (font (size 1.27 1.27)) (justify right))
     )
@@
       (project "OpenPowerDistribution"
         (path "/df87b081-37a2-452c-8581-7eff2c408a17/c5ef4c26-c64f-4464-8506-0cba199ca76f"
-          (reference "C56") (unit 1)
+          (reference "C5") (unit 1)
         )
       )
@@
         )
         (path "/df87b081-37a2-452c-8581-7eff2c408a17/c5ef4c26-c64f-4464-8506-0cba199ca76f"
-          (reference "C53") (unit 1)
+          (reference "C2") (unit 1)
         )
       )
@@
         )
         (path "/df87b081-37a2-452c-8581-7eff2c408a17/c5ef4c26-c64f-4464-8506-0cba199ca76f"
-          (reference "#PWR0157") (unit 1)
+          (reference "#PWR08") (unit 1)
         )
       )
@@
         )
         (path "/df87b081-37a2-452c-8581-7eff2c408a17/c5ef4c26-c64f-4464-8506-0cba199ca76f"
-          (reference "#PWR0155") (unit 1)
+          (reference "#PWR06") (unit 1)
         )
       )
@@
         )
         (path "/df87b081-37a2-452c-8581-7eff2c408a17/c5ef4c26-c64f-4464-8506-0cba199ca76f"
-          (reference "C55") (unit 1)
+          (reference "C4") (unit 1)
         )
       )
@@
   (symbol (lib_id "power:+5V") (at 170.18 76.2 0) (unit 1)
     (in_bom yes) (on_board yes) (dnp no) (fields_autoplaced)
-    (property "Reference" "#PWR0158" (at 170.18 80.01 0)
+    (property "Reference" "#PWR09" (at 170.18 80.01 0)
       (effects (font (size 1.27 1.27)) hide)
     )
@@
       (project "OpenPowerDistribution"
         (path "/df87b081-37a2-452c-8581-7eff2c408a17/c5ef4c26-c64f-4464-8506-0cba199ca76f"
-          (reference "#PWR0158") (unit 1)
+          (reference "#PWR09") (unit 1)
         )
       )
@@
         )
         (path "/df87b081-37a2-452c-8581-7eff2c408a17/c5ef4c26-c64f-4464-8506-0cba199ca76f"
-          (reference "U17") (unit 1)
-        )
-      )
+          (reference "U1") (unit 1)
+        )
+      )
