File: OpenPowerDistributor/Power input.kicad_sch (KiCad schematic)
At the start: 4 parts, among them J1 Barrel_Jack

Commit message: More schematic progress
Parts:
- removed C62: 330uF 25V, Capacitor_SMD:CP_Elec_8x10.5, symbol Device:CP_Small
- added C6: 47uF 16V, Capacitor_SMD:C_1210_3225Metric, symbol Device:C_Small
- J1: footprint (none) -> Connector_BarrelJack:BarrelJack_Horizontal
Connections:
- net +12V: now also C6.2
- net GND: now also C6.1
Changed lines of the file:
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@@
       (effects (font (size 1.27 1.27)))
     )
-    (property "Footprint" "" (at 135.89 91.186 0)
+    (property "Footprint" "Connector_BarrelJack:BarrelJack_Horizontal" (at 135.89 91.186 0)
       (effects (font (size 1.27 1.27)) hide)
     )
@@
     )
   )
-  (symbol (lib_id "Device:CP_Small") (at 185.42 92.71 0) (unit 1)
+  (symbol (lib_id "Device:C_Small") (at 185.42 92.71 180) (unit 1)
     (in_bom yes) (on_board yes) (dnp no)
-    (property "Reference" "C62" (at 187.6552 91.5416 0)
-      (effects (font (size 1.27 1.27)) (justify left))
+    (property "Reference" "C6" (at 187.96 91.4336 0)
+      (effects (font (size 1.27 1.27)) (justify right))
     )
-    (property "Value" "330uF 25V" (at 187.6552 93.853 0)
-      (effects (font (size 1.27 1.27)) (justify left))
+    (property "Value" "47uF 16V" (at 187.96 93.9736 0)
+      (effects (font (size 1.27 1.27)) (justify right))
     )
-    (property "Footprint" "Capacitor_SMD:CP_Elec_8x10.5" (at 185.42 92.71 0)
+    (property "Footprint" "Capacitor_SMD:C_1210_3225Metric" (at 185.42 92.71 0)
       (effects (font (size 1.27 1.27)) hide)
     )
@@
       (effects (font (size 1.27 1.27)) hide)
     )
-    (property "MPN" "GVT1E337M0810CNVC" (at 185.42 92.71 0)
+    (property "MPN" "CS3225X5R476K160NRL" (at 185.42 92.71 0)
+      (effects (font (size 1.27 1.27)) hide)
+    )
+    (property "LCSC Part#" "C2918513" (at 185.42 92.71 0)
       (effects (font (size 1.27 1.27)) hide)
     )
@@
     (pin "2")
     (instances
-      (project "KKS-Power-Board"
-        (path "/5f31b97b-d794-46d6-bbd9-7a5638bcf704/00000000-0000-0000-0000-000060e39742/32333c62-7f87-4aa0-b910-10a7c6d6b311"
-          (reference "C62") (unit 1)
+      (project "OpenPowerDistribution"
+        (path "/df87b081-37a2-452c-8581-7eff2c408a17/543a95e5-fa11-4cad-991c-06a5dbe63578"
+          (reference "C6") (unit 1)
         )
-        (path "/5f31b97b-d794-46d6-bbd9-7a5638bcf704/00000000-0000-0000-0000-000060e39742/43e6dee8-b6eb-4e16-bcb0-c3802573d004"
-          (reference "C56") (unit 1)
+        (path "/df87b081-37a2-452c-8581-7eff2c408a17/e80d9cb1-99ed-4151-affe-23d60cb9d8e2"
+          (reference "C55") (unit 1)
         )
-        (path "/5f31b97b-d794-46d6-bbd9-7a5638bcf704/00000000-0000-0000-0000-000060e39742/6708d228-a315-4a34-bc82-c41a553c79bb"
-          (reference "C68") (unit 1)
+        (path "/df87b081-37a2-452c-8581-7eff2c408a17/c5ef4c26-c64f-4464-8506-0cba199ca76f"
+          (reference "C55") (unit 1)
+        )
+        (path "/df87b081-37a2-452c-8581-7eff2c408a17/b2a621b0-638a-4528-852a-07ba08e58808"
+          (reference "C57") (unit 1)
         )
       )
-      (project "OpenPowerDistribution"
-        (path "/df87b081-37a2-452c-8581-7eff2c408a17/b2a621b0-638a-4528-852a-07ba08e58808"
-          (reference "C4") (unit 1)
-        )
-      )
