File: OpenPowerDistributor/Input multiplexer.kicad_sch (KiCad schematic)
At the start: 8 parts, among them U23 74HC165, U24 74HC165, U25 74HC165, U26 74HC165

Commit message: Analog multiplexer work
Connections:
- net +3.3V: now also C61.2, C61.2, U25.16 (VCC), U26.16 (VCC)
- net D_{In}10: no longer U26.13 (D2)
- net D_{In}11: no longer U26.14 (D3)
- net D_{In}12: no longer U26.3 (D4)
- net D_{In}13: no longer U26.4 (D5)
- net D_{In}14: no longer U26.5 (D6)
- net D_{In}15: no longer U26.6 (D7)
- net D_{In}8: no longer U26.11 (D0)
- net D_{In}9: no longer U26.12 (D1)
- new net D_{In}16: U26.11 (D0)
- new net D_{In}17: U26.12 (D1)
- new net D_{In}18: U26.13 (D2)
- new net D_{In}19: U26.14 (D3)
- new net D_{In}20: U26.3 (D4)
- new net D_{In}21: U26.4 (D5)
- new net D_{In}22: U26.5 (D6)
- new net D_{In}23: U26.6 (D7)
Changed lines of the file:
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@@
     (effects (font (size 1.27 1.27)) (justify left bottom))
   )
-  (label "D_{In}9" (at 143.466 134.62 0) (fields_autoplaced)
+  (label "D_{In}17" (at 143.466 134.62 0) (fields_autoplaced)
     (effects (font (size 1.27 1.27)) (justify left bottom))
   )
@@
     (effects (font (size 1.27 1.27)) (justify right bottom))
   )
-  (label "D_{In}13" (at 143.51 144.78 0) (fields_autoplaced)
+  (label "D_{In}21" (at 143.51 144.78 0) (fields_autoplaced)
     (effects (font (size 1.27 1.27)) (justify left bottom))
   )
@@
     (effects (font (size 1.27 1.27)) (justify right bottom))
   )
-  (label "D_{In}12" (at 143.51 142.24 0) (fields_autoplaced)
+  (label "D_{In}20" (at 143.51 142.24 0) (fields_autoplaced)
     (effects (font (size 1.27 1.27)) (justify left bottom))
   )
@@
     (effects (font (size 1.27 1.27)) (justify left bottom))
   )
-  (label "D_{In}11" (at 143.3659 139.7 0) (fields_autoplaced)
+  (label "D_{In}19" (at 143.3659 139.7 0) (fields_autoplaced)
     (effects (font (size 1.27 1.27)) (justify left bottom))
   )
@@
     (effects (font (size 1.27 1.27)) (justify right bottom))
   )
-  (label "D_{In}14" (at 143.51 147.32 0) (fields_autoplaced)
+  (label "D_{In}22" (at 143.51 147.32 0) (fields_autoplaced)
     (effects (font (size 1.27 1.27)) (justify left bottom))
   )
@@
     (effects (font (size 1.27 1.27)) (justify left bottom))
   )
-  (label "D_{In}8" (at 143.51 132.08 0) (fields_autoplaced)
+  (label "D_{In}16" (at 143.51 132.08 0) (fields_autoplaced)
     (effects (font (size 1.27 1.27)) (justify left bottom))
   )
@@
     (effects (font (size 1.27 1.27)) (justify left bottom))
   )
-  (label "D_{In}15" (at 143.51 149.86 0) (fields_autoplaced)
+  (label "D_{In}23" (at 143.51 149.86 0) (fields_autoplaced)
     (effects (font (size 1.27 1.27)) (justify left bottom))
   )
@@
     (effects (font (size 1.27 1.27)) (justify left bottom))
   )
-  (label "D_{In}10" (at 143.51 137.16 0) (fields_autoplaced)
+  (label "D_{In}18" (at 143.51 137.16 0) (fields_autoplaced)
     (effects (font (size 1.27 1.27)) (justify left bottom))
   )
@@
         (path "/df87b081-37a2-452c-8581-7eff2c408a17/d6281f85-5a0d-489c-bbcc-234cdb657621"
           (reference "#PWR0256") (unit 1)
+        )
+      )
+    )
+  )
+  (symbol (lib_id "power:+3.3V") (at 125.73 41.91 0) (unit 1)
+    (in_bom yes) (on_board yes) (dnp no) (fields_autoplaced)
+    (property "Reference" "#PWR0229" (at 125.73 45.72 0)
+      (effects (font (size 1.27 1.27)) hide)
+    )
+    (property "Value" "+3.3V" (at 125.73 38.1 0)
+      (effects (font (size 1.27 1.27)))
+    )
+    (property "Footprint" "" (at 125.73 41.91 0)
+      (effects (font (size 1.27 1.27)) hide)
+    )
+    (property "Datasheet" "" (at 125.73 41.91 0)
+      (effects (font (size 1.27 1.27)) hide)
+    )
+    (pin "1")
+    (instances
+      (project "OpenPowerDistribution"
+        (path "/df87b081-37a2-452c-8581-7eff2c408a17/5e66085e-4ac4-474e-a8c7-4febacc055ab"
+          (reference "#PWR0229") (unit 1)
+        )
+        (path "/df87b081-37a2-452c-8581-7eff2c408a17/d6281f85-5a0d-489c-bbcc-234cdb657621"
+          (reference "#PWR0274") (unit 1)
         )
       )
@@
         )
       )
+    )
+  )
+  (symbol (lib_id "power:+3.3V") (at 125.73 118.11 0) (unit 1)
+    (in_bom yes) (on_board yes) (dnp no) (fields_autoplaced)
+    (property "Reference" "#PWR0229" (at 125.73 121.92 0)
+      (effects (font (size 1.27 1.27)) hide)
+    )
+    (property "Value" "+3.3V" (at 125.73 114.3 0)
+      (effects (font (size 1.27 1.27)))
+    )
+    (property "Footprint" "" (at 125.73 118.11 0)
+      (effects (font (size 1.27 1.27)) hide)
+    )
+    (property "Datasheet" "" (at 125.73 118.11 0)
+      (effects (font (size 1.27 1.27)) hide)
+    )
+    (pin "1")
+    (instances
+      (project "OpenPowerDistribution"
+        (path "/df87b081-37a2-452c-8581-7eff2c408a17/5e66085e-4ac4-474e-a8c7-4febacc055ab"
+          (reference "#PWR0229") (unit 1)
+        )
+        (path "/df87b081-37a2-452c-8581-7eff2c408a17/d6281f85-5a0d-489c-bbcc-234cdb657621"
+          (reference "#PWR0275") (unit 1)
+        )
+      )
