File: OpenPowerDistributor/Output channels.kicad_sch (KiCad schematic)
At the start: 18 parts

Commit message: Analog multiplexer work
Changed lines of the file:
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@@
     (effects (font (size 1.27 1.27)) (justify left bottom))
   )
-  (label "A_{In}2" (at 109.22 93.98 0) (fields_autoplaced)
+  (label "A_{In}12" (at 109.22 134.62 0) (fields_autoplaced)
     (effects (font (size 1.27 1.27)) (justify left bottom))
   )
@@
     (effects (font (size 1.27 1.27)) (justify left bottom))
   )
-  (label "A_{In}4" (at 31.75 156.21 0) (fields_autoplaced)
+  (label "A_{In}6" (at 31.75 156.21 0) (fields_autoplaced)
     (effects (font (size 1.27 1.27)) (justify left bottom))
   )
@@
     (effects (font (size 1.27 1.27)) (justify left bottom))
   )
-  (label "A_{In}1" (at 109.22 125.73 0) (fields_autoplaced)
+  (label "A_{In}9" (at 109.22 85.09 0) (fields_autoplaced)
     (effects (font (size 1.27 1.27)) (justify left bottom))
   )
@@
     (effects (font (size 1.27 1.27)) (justify left bottom))
   )
-  (label "A_{In}1" (at 109.22 85.09 0) (fields_autoplaced)
+  (label "A_{In}11" (at 109.22 125.73 0) (fields_autoplaced)
     (effects (font (size 1.27 1.27)) (justify left bottom))
   )
@@
     (effects (font (size 1.27 1.27)) (justify left bottom))
   )
-  (label "A_{In}1" (at 109.22 168.91 0) (fields_autoplaced)
+  (label "A_{In}7" (at 109.22 34.29 0) (fields_autoplaced)
     (effects (font (size 1.27 1.27)) (justify left bottom))
   )
@@
     (effects (font (size 1.27 1.27)) (justify left bottom))
   )
-  (label "A_{In}3" (at 31.75 147.32 0) (fields_autoplaced)
-    (effects (font (size 1.27 1.27)) (justify left bottom))
-  )
-  (label "A_{In}2" (at 109.22 134.62 0) (fields_autoplaced)
+  (label "A_{In}5" (at 31.75 147.32 0) (fields_autoplaced)
+    (effects (font (size 1.27 1.27)) (justify left bottom))
+  )
+  (label "A_{In}10" (at 109.22 93.98 0) (fields_autoplaced)
     (effects (font (size 1.27 1.27)) (justify left bottom))
   )
@@
     (effects (font (size 1.27 1.27)) (justify left bottom))
   )
-  (label "A_{In}2" (at 185.42 85.09 0) (fields_autoplaced)
+  (label "A_{In}16" (at 185.42 85.09 0) (fields_autoplaced)
     (effects (font (size 1.27 1.27)) (justify left bottom))
   )
@@
     (effects (font (size 1.27 1.27)) (justify left bottom))
   )
-  (label "A_{In}2" (at 185.42 128.27 0) (fields_autoplaced)
+  (label "A_{In}18" (at 185.42 128.27 0) (fields_autoplaced)
     (effects (font (size 1.27 1.27)) (justify left bottom))
   )
@@
     (effects (font (size 1.27 1.27)) (justify left bottom))
   )
-  (label "A_{In}1" (at 109.22 34.29 0) (fields_autoplaced)
+  (label "A_{In}13" (at 109.22 168.91 0) (fields_autoplaced)
     (effects (font (size 1.27 1.27)) (justify left bottom))
   )
@@
     (effects (font (size 1.27 1.27)) (justify left bottom))
   )
-  (label "A_{In}1" (at 185.42 119.38 0) (fields_autoplaced)
+  (label "A_{In}17" (at 185.42 119.38 0) (fields_autoplaced)
     (effects (font (size 1.27 1.27)) (justify left bottom))
   )
@@
     (effects (font (size 1.27 1.27)) (justify left bottom))
   )
-  (label "A_{In}1" (at 185.42 76.2 0) (fields_autoplaced)
+  (label "A_{In}15" (at 185.42 76.2 0) (fields_autoplaced)
     (effects (font (size 1.27 1.27)) (justify left bottom))
   )
@@
     (effects (font (size 1.27 1.27)) (justify left bottom))
   )
-  (label "A_{In}2" (at 109.22 177.8 0) (fields_autoplaced)
+  (label "A_{In}8" (at 109.22 43.18 0) (fields_autoplaced)
     (effects (font (size 1.27 1.27)) (justify left bottom))
   )
@@
     (effects (font (size 1.27 1.27)) (justify left bottom))
   )
-  (label "A_{In}2" (at 109.22 43.18 0) (fields_autoplaced)
-    (effects (font (size 1.27 1.27)) (justify left bottom))
-  )
+  (label "A_{In}14" (at 109.22 177.8 0) (fields_autoplaced)
+    (effects (font (size 1.27 1.27)) (justify left bottom))
+  )
