File: OpenPowerDistributor/Output multiplexer.kicad_sch (KiCad schematic)
At the start: 15 parts, among them U10 74HCT595, U11 74HCT595, U12 74HCT595, U13 74HCT595, U14 74HCT595, U15 74HCT595

Commit message: Start to make layout
Parts:
- renumbered C28 to C61, C29 to C62, C30 to C63, C31 to C64, C32 to C65, C33 to C66, C33 to C67, R39 to R225, U10 to U16, U11 to U17, U12 to U18, U13 to U19, U14 to U20, U15 to U21, U15 to U22
Connections:
- net MUX-IO0 renamed D_{Out}0
- net MUX-IO1 renamed D_{Out}1
- net MUX-IO10 renamed D_{Out}10
- net MUX-IO11 renamed D_{Out}11
- net MUX-IO12 renamed D_{Out}12
- net MUX-IO13 renamed D_{Out}13
- net MUX-IO14 renamed D_{Out}14
- net MUX-IO15 renamed D_{Out}15
- net MUX-IO16 renamed D_{Out}16
- net MUX-IO17 renamed D_{Out}17
- net MUX-IO18 renamed D_{Out}18
- net MUX-IO19 renamed D_{Out}19
- net MUX-IO2 renamed D_{Out}2
- net MUX-IO20 renamed D_{Out}20
- net MUX-IO21 renamed D_{Out}21
- net MUX-IO22 renamed D_{Out}22
- net MUX-IO23 renamed D_{Out}23
- net MUX-IO24 renamed D_{Out}24
- net MUX-IO25 renamed D_{Out}25
- net MUX-IO26 renamed D_{Out}26
- net MUX-IO27 renamed D_{Out}27
- net MUX-IO28 renamed D_{Out}28
- net MUX-IO29 renamed D_{Out}29
- net MUX-IO3 renamed D_{Out}3
- net MUX-IO30 renamed D_{Out}30
- net MUX-IO31 renamed D_{Out}31
- net MUX-IO32 renamed D_{Out}32
- net MUX-IO33 renamed D_{Out}33
- net MUX-IO34 renamed D_{Out}34
- net MUX-IO35 renamed D_{Out}35
- net MUX-IO36 renamed D_{Out}36
- net MUX-IO37 renamed D_{Out}37
- net MUX-IO38 renamed D_{Out}38
- net MUX-IO39 renamed D_{Out}39
- net MUX-IO4 renamed D_{Out}4
- net MUX-IO40 renamed D_{Out}40
- net MUX-IO41 renamed D_{Out}41
- net MUX-IO42 renamed D_{Out}42
- net MUX-IO43 renamed D_{Out}43
- net MUX-IO44 renamed D_{Out}44
- net MUX-IO45 renamed D_{Out}45
- net MUX-IO46 renamed D_{Out}46
- net MUX-IO47 renamed D_{Out}47
- net MUX-IO48 renamed D_{Out}48
- net MUX-IO49 renamed D_{Out}49
- net MUX-IO5 renamed D_{Out}5
- net MUX-IO50 renamed D_{Out}50
- net MUX-IO51 renamed D_{Out}51
- net MUX-IO52 renamed D_{Out}52
- net MUX-IO53 renamed D_{Out}53
- net MUX-IO54 renamed D_{Out}54
- net MUX-IO55 renamed D_{Out}55
- net MUX-IO6 renamed D_{Out}6
- net MUX-IO7 renamed D_{Out}7
- net MUX-IO8 renamed D_{Out}8
- net MUX-IO9 renamed D_{Out}9
Other:
- note added: "Normally-keep MUX-LOAD low. After loading data in the registers, run a single HIGH pulse on LOAD"
- note removed: "Normally-keep Reg-LOAD low. After loading data in the registers, run a single HIGH pulse on LOAD"
