File: OpenPowerDistributor/Analog multiplexer.kicad_sch (KiCad schematic)
At the start: 4 parts, among them U27 CD4067BMT/TR, U28 CD4067BMT/TR

Commit message: Work mostly on Ethernet schematic
Connections:
- net AIN2 is gone; now on net AMUX-Out: U28.1 (COM)
- net AIN1 renamed AMUX-Out
Changed lines of the file:
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@@
 (kicad_sch (version 20230121) (generator eeschema)
   (paper "A4")
+  (junction (at 128.27 43.18) (diameter 0) (color 0 0 0 0)
+  )
   (bus_entry (at 130.81 58.42) (size 2.54 -2.54)
     (stroke (width 0) (type default))
@@
     (stroke (width 0) (type default))
   )
+  (wire (pts (xy 125.73 43.18) (xy 128.27 43.18))
+    (stroke (width 0) (type default))
+  )
   (bus (pts (xy 90.17 31.75) (xy 130.81 31.75))
     (stroke (width 0) (type default))
@@
     (stroke (width 0) (type default))
   )
+  (wire (pts (xy 128.27 113.03) (xy 153.67 113.03))
+    (stroke (width 0) (type default))
+  )
   (bus (pts (xy 130.81 130.81) (xy 130.81 133.35))
+    (stroke (width 0) (type default))
+  )
+  (wire (pts (xy 128.27 43.18) (xy 153.67 43.18))
     (stroke (width 0) (type default))
   )
@@
   )
   (wire (pts (xy 133.35 58.42) (xy 153.67 58.42))
+    (stroke (width 0) (type default))
+  )
+  (wire (pts (xy 128.27 43.18) (xy 128.27 113.03))
     (stroke (width 0) (type default))
   )
@@
     (effects (font (size 1.27 1.27)) (justify right bottom))
   )
-  (hierarchical_label "AIN2" (shape input) (at 153.67 113.03 180) (fields_autoplaced)
+  (hierarchical_label "AMUX-Out" (shape output) (at 125.73 43.18 180) (fields_autoplaced)
     (effects (font (size 1.27 1.27)) (justify right))
   )
-  (hierarchical_label "AIN1" (shape input) (at 153.67 43.18 180) (fields_autoplaced)
-    (effects (font (size 1.27 1.27)) (justify right))
-  )
