File: OpenPowerDistributor/OpenPowerDistribution.kicad_pcb (KiCad board)
At the start: 2 copper layers, 478 parts, among them J1 Barrel_Jack, J10 Barrel_Jack, J11 Barrel_Jack, J12 Barrel_Jack, J13 Barrel_Jack, J14 Barrel_Jack, J15 Barrel_Jack, J16 Barrel_Jack, J17 Barrel_Jack, J18 Barrel_Jack, J19 Barrel_Jack, J2 Barrel_Jack, J3 Barrel_Jack, J4 Barrel_Jack, J5 Barrel_Jack, J6 Barrel_Jack, J7 Barrel_Jack, J8 Barrel_Jack, J9 Barrel_Jack, Q1 BC847, Q10 BC847, Q11 STN2610D, Q12 STN2610D, Q13 BC847, Q14 BC847, Q15 BC847, Q16 BC847, Q17 STN2610D, Q18 STN2610D, Q19 BC847, Q2 BC847, Q20 BC847, Q21 BC847, Q22 BC847, Q23 STN2610D, Q24 STN2610D, Q25 BC847, Q26 BC847, Q27 BC847, Q28 BC847, Q29 STN2610D, Q3 BC847, Q30 STN2610D, Q31 BC847, Q32 BC847, Q33 BC847, Q34 BC847, Q35 STN2610D, Q36 STN2610D, Q37 BC847, Q38 BC847, Q39 BC847, Q4 BC847, Q40 BC847, Q41 STN2610D, Q42 STN2610D, Q43 BC847, Q44 BC847, Q45 BC847, Q46 BC847, Q47 STN2610D, Q48 STN2610D, Q49 BC847, Q5 STN2610D, Q50 BC847, Q51 BC847, Q52 BC847, Q53 STN2610D, Q54 STN2610D, Q6 STN2610D, Q7 BC847, Q8 BC847, Q9 BC847, U1 AP63200WU, U10 LM324, U11 LM324, U12 LM324, U13 LM324, U17 TPS565208DDA, U18 TPS565208DDA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

Commit message: Start to make layout
Parts:
- removed the U13 at (139.9, 36.0)
- added C61: 100nF, Capacitor_SMD:C_0603_1608Metric, F.Cu at (48.5, -6.36)
- added C62: 100nF, Capacitor_SMD:C_0603_1608Metric, F.Cu at (48.5, -3.85)
- added C63: 100nF, Capacitor_SMD:C_0603_1608Metric, F.Cu at (48.5, -1.33)
- added C64: 100nF, Capacitor_SMD:C_0603_1608Metric, F.Cu at (48.5, 1.18)
- added C65: 100nF, Capacitor_SMD:C_0603_1608Metric, F.Cu at (48.5, 3.69)
- added C66: 100nF, Capacitor_SMD:C_0603_1608Metric, F.Cu at (48.5, 6.20)
- added C67: 100nF, Capacitor_SMD:C_0603_1608Metric, F.Cu at (48.5, 8.71)
- added C68: 100nF, Capacitor_SMD:C_0603_1608Metric, F.Cu at (21.7, 15.0)
- added C69: 100nF, Capacitor_SMD:C_0603_1608Metric, F.Cu at (11.7, 2.06)
- added C70: 100nF, Capacitor_SMD:C_0603_1608Metric, F.Cu at (11.7, 4.57)
- added C71: 100nF, Capacitor_SMD:C_0603_1608Metric, F.Cu at (11.7, 7.08)
- added FB10: 220R@100MHz 3A, Inductor_SMD:L_0805_2012Metric, F.Cu at (53.1, 143.4)
- added FB11: 220R@100MHz 3A, Inductor_SMD:L_0805_2012Metric, F.Cu at (119.3, -32.7)
- added FB12: 220R@100MHz 3A, Inductor_SMD:L_0805_2012Metric, F.Cu at (112.8, -32.7)
- added FB13: 220R@100MHz 3A, Inductor_SMD:L_0805_2012Metric, F.Cu at (119.3, -42.2)
- added FB14: 220R@100MHz 3A, Inductor_SMD:L_0805_2012Metric, F.Cu at (112.8, -42.2)
- added FB15: 220R@100MHz 3A, Inductor_SMD:L_0805_2012Metric, F.Cu at (106.2, -42.2)
- added FB16: 220R@100MHz 3A, Inductor_SMD:L_0805_2012Metric, F.Cu at (106.2, -32.7)
- added FB17: 220R@100MHz 3A, Inductor_SMD:L_0805_2012Metric, F.Cu at (106.2, -37.5)
- added FB18: 220R@100MHz 3A, Inductor_SMD:L_0805_2012Metric, F.Cu at (119.3, -37.5)
- added R225: 220k, Resistor_SMD:R_0603_1608Metric, F.Cu at (48.5, 11.2)
- added U16: 74HCT595, Package_SO:TSSOP-16_4.4x5mm_P0.65mm, F.Cu at (42.1, -4.32)
- added U17: 74HCT595, Package_SO:TSSOP-16_4.4x5mm_P0.65mm, F.Cu at (42.1, 2.27)
- added U18: 74HCT595, Package_SO:TSSOP-16_4.4x5mm_P0.65mm, F.Cu at (42.1, 8.87)
- added U19: 74HCT595, Package_SO:TSSOP-16_4.4x5mm_P0.65mm, F.Cu at (42.1, 15.5)
- added U20: 74HCT595, Package_SO:TSSOP-16_4.4x5mm_P0.65mm, F.Cu at (42.1, 22.0)
- added U21: 74HCT595, Package_SO:TSSOP-16_4.4x5mm_P0.65mm, F.Cu at (42.1, 28.6)
- added U22: 74HCT595, Package_SO:TSSOP-16_4.4x5mm_P0.65mm, F.Cu at (42.1, 35.2)
- added U23: 74HC165, Package_SO:TSSOP-16_4.4x5mm_P0.65mm, F.Cu at (15.3, 12.6)
- added U24: 74HC165, Package_SO:TSSOP-16_4.4x5mm_P0.65mm, F.Cu at (5.36, 4.09)
- added U25: 74HC165, Package_SO:TSSOP-16_4.4x5mm_P0.65mm, F.Cu at (5.36, 10.7)
- added U26: 74HC165, Package_SO:TSSOP-16_4.4x5mm_P0.65mm, F.Cu at (5.36, 17.3)
- moved D10 248.2 mm to (23.0, 167.6), turned to 90 degrees
- moved D9 246.4 mm to (34.6, 167.3), turned to 90 degrees
- moved R23 239.3 mm to (35.2, 153.5), turned to 90 degrees
- moved J2 236.2 mm to (29.0, 155.0), turned to 90 degrees
- moved R24 229.9 mm to (55.2, 153.2), turned to 90 degrees
- moved D5 227.4 mm to (38.2, 152.1), turned to 90 degrees
- moved FB1 224.5 mm to (33.5, 143.5), turned to -90 degrees
- moved D6 222.2 mm to (42.0, 152.1), turned to 90 degrees
- moved R28 220.3 mm to (23.0, 164.6), turned to 90 degrees
- moved R27 218.2 mm to (34.6, 164.2), turned to 90 degrees
- moved J3 218.2 mm to (49.0, 155.0), turned to 90 degrees
- moved D7 217.7 mm to (28.8, 139.8), turned to 180 degrees
- moved U4 217.4 mm to (39.9, 141.9), turned to 90 degrees
- moved Q3 217.0 mm to (38.2, 159.3), turned to 90 degrees
- moved R9 215.6 mm to (31.5, 136.1), turned to 90 degrees
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- renumbered C57 to C1, C7 to C10, C6 to C11, C33 to C12, C34 to C13, C35 to C14, C36 to C15, C37 to C16, C8 to C17, C9 to C18, C10 to C19, C53 to C2, C11 to C20, C12 to C21, C13 to C22, C14 to C23, C15 to C24, C16 to C25, C17 to C26, C23 to C27, C24 to C28, C25 to C29, C54 to C3, C26 to C30, C27 to C31, C28 to C32, C29 to C33, C30 to C34, C31 to C35, C32 to C36, C38 to C37, C39 to C38, C40 to C39, C55 to C4, C41 to C40, C42 to C41, C18 to C42, C19 to C43, C20 to C44, C21 to C45, C22 to C46, C4 to C47, C58 to C48, C59 to C49, C43 to C51, C44 to C52, C45 to C53, C46 to C54, C47 to C55, C48 to C56, C49 to C57, C50 to C58, C51 to C59, C1 to C6, C52 to C60, C2 to C7, C3 to C8, C5 to C9, D44 to D10, D41 to D11, D42 to D12, D5 to D13, D6 to D14, D7 to D15, D8 to D16, D9 to D17, D10 to D18, D11 to D19, D12 to D20, D15 to D21, D16 to D22, D17 to D23, D18 to D24, D19 to D25, D20 to D26, D21 to D27, D22 to D28, D33 to D29, D34 to D30, D35 to D31, D36 to D32, D45 to D33, D46 to D34, D47 to D35, D48 to D36, D49 to D37, D50 to D38, D51 to D39, D52 to D40, D53 to D41, D54 to D42, D55 to D43, D56 to D44, D59 to D45, D60 to D46, D61 to D47, D62 to D48, D63 to D49, D37 to D5, D64 to D50, D65 to D51, D66 to D52, D25 to D53, D26 to D54, D27 to D55, D28 to D56, D29 to D57, D30 to D58, D31 to D59, D38 to D6, D32 to D60, D69 to D61, D70 to D62, D71 to D63, D72 to D64, D73 to D65, D74 to D66, D75 to D67, D76 to D68, D85 to D69, D39 to D7, D86 to D70, D13 to D71, D14 to D72, D23 to D73, D24 to D74, D77 to D75, D78 to D76, D79 to D77, D80 to D78, D57 to D79, D40 to D8, D58 to D80, D67 to D81, D68 to D82, D91 to D83, D92 to D84, D93 to D85, D94 to D86, D81 to D87, D82 to D88, D83 to D89, D43 to D9, D84 to D90, D87 to D91, D88 to D92, D89 to D93, D90 to D94, FB5 to FB4, FB6 to FB5, FB7 to FB6, FB4 to FB7, J14 to J12, J15 to J13, J6 to J14, J7 to J15, J12 to J2, J13 to J3, J2 to J4, J3 to J5, J4 to J6, J5 to J7, L3 to L1, L1 to L2, L2 to L3, Q31 to Q1, Q4 to Q10, Q5 to Q11, Q6 to Q12, Q7 to Q13, Q8 to Q14, Q9 to Q15, Q10 to Q16, Q11 to Q17, Q12 to Q18, Q32 to Q2, Q33 to Q3, Q37 to Q31, Q38 to Q32, Q39 to Q33, Q40 to Q34, Q41 to Q35, Q42 to Q36, Q13 to Q37, Q14 to Q38, Q15 to Q39, Q34 to Q4, Q16 to Q40, Q17 to Q41, Q18 to Q42, Q35 to Q5, Q36 to Q6, Q1 to Q7, Q2 to Q8, Q3 to Q9, R167 to R1, R6 to R10, R122 to R100, R123 to R101, R124 to R102, R125 to R103, R126 to R104, R127 to R105, R128 to R106, R129 to R107, R130 to R108, R131 to R109, R102 to R11, R132 to R110, R133 to R111, R134 to R112, R135 to R113, R136 to R114, R137 to R115, R138 to R116, R139 to R117, R140 to R118, R141 to R119, R101 to R12, R142 to R120, R143 to R121, R144 to R122, R145 to R123, R146 to R124, R147 to R125, R148 to R126, R149 to R127, R150 to R128, R151 to R129, R103 to R13, R152 to R130, R153 to R131, R154 to R132, R155 to R133, R156 to R134, R157 to R135, R158 to R136, R159 to R137, R160 to R138, R161 to R139, R104 to R14, R162 to R140, R163 to R141, R164 to R142, R165 to R143, R166 to R144, R171 to R145, R172 to R146, R173 to R147, R174 to R148, R175 to R149, R105 to R15, R176 to R150, R55 to R151, R56 to R152, R57 to R153, R58 to R154, R59 to R155, R60 to R156, R61 to R157, R62 to R158, R63 to R159, R106 to R16, R64 to R160, R65 to R161, R66 to R162, R67 to R163, R68 to R164, R69 to R165, R70 to R166, R71 to R167, R72 to R168, R73 to R169, R107 to R17, R74 to R170, R75 to R171, R76 to R172, R77 to R173, R78 to R174, R169 to R175, R170 to R176, R108 to R18, R109 to R19, R168 to R2, R110 to R20, R111 to R21, R112 to R22, R113 to R23, R114 to R24, R115 to R25, R116 to R26, R119 to R27, R120 to R28, R117 to R29, R1 to R3, R118 to R30, R7 to R31, R8 to R32, R9 to R33, R10 to R34, R11 to R35, R12 to R36, R13 to R37, R14 to R38, R15 to R39, R2 to R4, R16 to R40, R17 to R41, R18 to R42, R19 to R43, R20 to R44, R21 to R45, R22 to R46, R23 to R47, R24 to R48, R25 to R49, R3 to R5, R26 to R50, R27 to R51, R28 to R52, R29 to R53, R30 to R54, R31 to R55, R32 to R56, R33 to R57, R34 to R58, R35 to R59, R4 to R6, R36 to R60, R37 to R61, R38 to R62, R39 to R63, R40 to R64, R41 to R65, R42 to R66, R43 to R67, R44 to R68, R45 to R69, R99 to R7, R46 to R70, R47 to R71, R48 to R72, R49 to R73, R50 to R74, R51 to R75, R52 to R76, R53 to R77, R54 to R78, R100 to R8, R5 to R9, R121 to R99, U17 to U1, U7 to U10, U9 to U11, U6 to U12, U18 to U13, U3 to U15, U1 to U2, U2 to U3, U8 to U4, U10 to U5, U11 to U6, U12 to U7, U4 to U8, U5 to U9
Connections:
- C13 pad 1: Net-(U10C-+) (its old number) -> Net-(U4C-+)
- C13 pad 2: Net-(C34-Pad2) -> Net-(C13-Pad2)
- C14 pad 1: Net-(U11B--) -> Net-(U4B--)
- C15 pad 1: Net-(U12D--) (its old number) -> Net-(U4D--)
- C33 pad 1: Net-(U8C-+) (its old number) -> Net-(U11C-+)
- C33 pad 2: Net-(C29-Pad2) -> Net-(C33-Pad2)
- C34 pad 1: Net-(U8B--) (its old number) -> Net-(U11B--)
- C35 pad 1: Net-(U8D--) (its old number) -> Net-(U11D--)
- C38 pad 1: Net-(U9C-+) (its old number) -> Net-(U5C-+)
- C38 pad 2: Net-(C39-Pad2) -> Net-(C38-Pad2)
- C39 pad 1: Net-(U9B--) (its old number) -> Net-(U5B--)
- C40 pad 1: Net-(U9D--) (its old number) -> Net-(U5D--)
- C53 pad 1: Net-(U10B--) (its old number) -> Net-(U6B--)
- C54 pad 1: Net-(U10D--) (its old number) -> Net-(U6D--)
- C58 pad 1: Net-(U13B--) -> Net-(U7B--)
- C59 pad 1: Net-(U13D--) -> Net-(U7D--)
- D16 pad 1: Net-(D8-K) -> Net-(D16-K)
- D24 pad 1: Net-(D18-K) -> Net-(D24-K)
- D32 pad 1: Net-(D36-K) -> Net-(D32-K)
- D40 pad 1: Net-(D52-K) -> Net-(D40-K)
- D48 pad 1: Net-(D62-K) -> Net-(D48-K)
- D56 pad 1: Net-(D28-K) -> Net-(D56-K)
- D64 pad 1: Net-(D72-K) -> Net-(D64-K)
- D8 pad 1: Net-(D40-K) -> Net-(D8-K)
- D90 pad 1: Net-(D84-K) -> Net-(D90-K)
- Q12 pad 2: Net-(D8-K) -> Net-(Q12-D)
- Q18 pad 2: Net-(D18-K) -> Net-(Q18-D)
- Q24 pad 2: Net-(D36-K) -> Net-(Q24-D)
- Q30 pad 2: Net-(D52-K) -> Net-(Q30-D)
- Q36 pad 2: Net-(D62-K) -> Net-(Q36-D)
- Q42 pad 2: Net-(D28-K) -> Net-(Q42-D)
- Q48 pad 2: Net-(D72-K) -> Net-(Q48-D)
- Q54 pad 2: Net-(D84-K) -> Net-(Q54-D)
- Q6 pad 2: Net-(D40-K) -> Net-(Q6-D)
- R104 pad 2: Net-(U8C-+) (its old number) -> Net-(U11C-+)
- R107 pad 2: Net-(C29-Pad2) -> Net-(C33-Pad2)
- R11 pad 2: Net-(C34-Pad2) -> Net-(C13-Pad2)
- R110 pad 1: Net-(C29-Pad2) -> Net-(C33-Pad2)
- R115 pad 2: Net-(U8B--) (its old number) -> Net-(U11B--)
- R116 pad 2: Net-(U8D--) (its old number) -> Net-(U11D--)
- R117 pad 2: Net-(U8B--) (its old number) -> Net-(U11B--)
- R118 pad 2: Net-(U8D--) (its old number) -> Net-(U11D--)
- R128 pad 2: Net-(U9C-+) (its old number) -> Net-(U5C-+)
- R131 pad 2: Net-(C39-Pad2) -> Net-(C38-Pad2)
- R134 pad 1: Net-(C39-Pad2) -> Net-(C38-Pad2)
- R139 pad 2: Net-(U9B--) (its old number) -> Net-(U5B--)
- R14 pad 1: Net-(C34-Pad2) -> Net-(C13-Pad2)
- R140 pad 2: Net-(U9D--) (its old number) -> Net-(U5D--)
- R141 pad 2: Net-(U9B--) (its old number) -> Net-(U5B--)
- R142 pad 2: Net-(U9D--) (its old number) -> Net-(U5D--)
- R189 pad 2: Net-(U10B--) (its old number) -> Net-(U6B--)
- R19 pad 2: Net-(U11B--) -> Net-(U4B--)
- R190 pad 2: Net-(U10D--) (its old number) -> Net-(U6D--)
- R191 pad 2: Net-(U10B--) (its old number) -> Net-(U6B--)
- R192 pad 2: Net-(U10D--) (its old number) -> Net-(U6D--)
- R20 pad 2: Net-(U12D--) (its old number) -> Net-(U4D--)
- R21 pad 2: Net-(U11B--) -> Net-(U4B--)
- R213 pad 2: Net-(U13B--) -> Net-(U7B--)
- R214 pad 2: Net-(U13D--) -> Net-(U7D--)
- R215 pad 2: Net-(U13B--) -> Net-(U7B--)
- R216 pad 2: Net-(U13D--) -> Net-(U7D--)
- R22 pad 2: Net-(U12D--) (its old number) -> Net-(U4D--)
- R8 pad 2: Net-(U10C-+) (its old number) -> Net-(U4C-+)
- U11 pad 10: Net-(U9C-+) (its old number) -> Net-(U11C-+)
- U11 pad 12: /DC Output channels/12V output #3/O2+ -> /DC Output channels/12V output #2/O2+
- U11 pad 13: Net-(U9D--) (its old number) -> Net-(U11D--)
- U11 pad 5: /DC Output channels/12V output #3/O1- -> /DC Output channels/12V output #2/O1-
- U11 pad 6: Net-(U9B--) (its old number) -> Net-(U11B--)
- U11 pad 8: Net-(C39-Pad2) -> Net-(C33-Pad2)
- U4 pad 10: Net-(U8C-+) (its old number) -> Net-(U4C-+)
- U4 pad 12: /DC Output channels/12V output #2/O2+ -> /DC Output channels/5V output #1/O2+
- U4 pad 13: Net-(U8D--) (its old number) -> Net-(U4D--)
- U4 pad 5: /DC Output channels/12V output #2/O1- -> /DC Output channels/5V output #1/O1-
- U4 pad 6: Net-(U8B--) (its old number) -> Net-(U4B--)
- U4 pad 8: Net-(C29-Pad2) -> Net-(C13-Pad2)
- U5 pad 10: Net-(U10C-+) (its old number) -> Net-(U5C-+)
- U5 pad 12: /DC Output channels/9V output #1/O2+ -> /DC Output channels/12V output #3/O2+
- U5 pad 13: Net-(U10D--) (its old number) -> Net-(U5D--)
- U5 pad 5: /DC Output channels/9V output #1/O1- -> /DC Output channels/12V output #3/O1-
- U5 pad 6: Net-(U10B--) (its old number) -> Net-(U5B--)
- U5 pad 8: Net-(C34-Pad2) -> Net-(C38-Pad2)
- U6 pad 12: (no net) -> /DC Output channels/9V output #1/O2+
- U6 pad 13: (no net) -> Net-(U6D--)
- U6 pad 14: (no net) -> /DC Output channels/A_{In}2
- U6 pad 5: /DC Output channels/5V output #1/O1- -> /DC Output channels/9V output #1/O1-
- U6 pad 6: Net-(U11B--) -> Net-(U6B--)
- U7 pad 12: /DC Output channels/5V output #1/O2+ -> /DC Output channels/9V output #2/O2+
- U7 pad 13: Net-(U12D--) (its old number) -> Net-(U7D--)
- U7 pad 5: (no net) -> /DC Output channels/9V output #2/O1-
- U7 pad 6: (no net) -> Net-(U7B--)
- U7 pad 7: (no net) -> /DC Output channels/A_{In}1

Commit message: Analog multiplexer work
Parts:
- added D95: SS36(F), Diode_SMD:D_SMA, F.Cu at (38.6, -27.9)
- added J20: USB_C_Receptacle_USB2.0, Connector_USB:USB_C_Receptacle_HCTL_HC-TYPE-C-16P-01A, F.Cu at (49.9, -26.3)
- added R226: 10k, Resistor_SMD:R_0603_1608Metric, F.Cu at (46.0, -43.0)
- added R227: 5.1k, Resistor_SMD:R_0603_1608Metric, F.Cu at (46.0, -40.5)
- added R228: 5.1k, Resistor_SMD:R_0603_1608Metric, F.Cu at (46.0, -38.0)
- added R229: 10k, Resistor_SMD:R_0603_1608Metric, F.Cu at (46.0, -35.5)
- added R230: 10k, Resistor_SMD:R_0603_1608Metric, F.Cu at (46.0, -33.0)
- added SW1: RST, Button_Switch_SMD:SW_SPST_TL3342, F.Cu at (39.3, -40.7)
- added SW2: BOOT, Button_Switch_SMD:SW_SPST_TL3342, F.Cu at (39.3, -33.7)
- added U14: USBLC6-2SC6, Package_TO_SOT_SMD:SOT-23-6, F.Cu at (50.6, -42.0)
Connections:
- C70 pad 2: Net-(U25-VCC) -> +3.3V
- C71 pad 2: Net-(U26-VCC) -> +3.3V
- U15 pad 22: unconnected-(U15-USB_D--Pad22) -> /MCU/USB-D-
- U15 pad 23: unconnected-(U15-USB_D+-Pad23) -> /MCU/USB-D+
- U15 pad 3: unconnected-(U15-IO00-Pad3) -> Net-(U15-IO00)
- U15 pad 41: unconnected-(U15-EN-Pad41) -> ESP32-~{RST}
- U15 pad 5: unconnected-(U15-IO02-Pad5) -> Net-(U15-IO02)
- U25 pad 16: Net-(U25-VCC) -> +3.3V
- U26 pad 11: /Input multiplexer/D_{In}8 -> /Input multiplexer/D_{In}16
- U26 pad 12: /Input multiplexer/D_{In}9 -> /Input multiplexer/D_{In}17
- U26 pad 13: /Input multiplexer/D_{In}10 -> /Input multiplexer/D_{In}18
- U26 pad 14: /Input multiplexer/D_{In}11 -> /Input multiplexer/D_{In}19
- U26 pad 16: Net-(U26-VCC) -> +3.3V
- U26 pad 3: /Input multiplexer/D_{In}12 -> /Input multiplexer/D_{In}20
- U26 pad 4: /Input multiplexer/D_{In}13 -> /Input multiplexer/D_{In}21
- U26 pad 5: /Input multiplexer/D_{In}14 -> /Input multiplexer/D_{In}22
- U26 pad 6: /Input multiplexer/D_{In}15 -> /Input multiplexer/D_{In}23

Commit message: Work mostly on Ethernet schematic
Parts:
- removed D95: SS36(F), Diode_SMD:D_SMA
- removed SW2: BOOT, Button_Switch_SMD:SW_SPST_TL3342
- added C72: 100nF 16V, Capacitor_SMD:C_0603_1608Metric, F.Cu at (-49.0, 30.4)
- added C73: 100nF 16V, Capacitor_SMD:C_0603_1608Metric, F.Cu at (-49.0, 32.9)
- added C74: 100nF, Capacitor_SMD:C_0603_1608Metric, F.Cu at (-103.0, 66.3)
- added C75: 100nF, Capacitor_SMD:C_0603_1608Metric, F.Cu at (-55.0, -9.29)
- added C76: 1uF 6.3V, Capacitor_SMD:C_0603_1608Metric, F.Cu at (-55.0, -6.79)
- added C77: 100nF, Capacitor_SMD:C_0603_1608Metric, F.Cu at (-55.0, -4.28)
- added C78: 100nF, Capacitor_SMD:C_0603_1608Metric, F.Cu at (-55.0, -1.76)
- added C79: 1uF 6.3V, Capacitor_SMD:C_0603_1608Metric, F.Cu at (-72.6, 21.2)
- added C81: 100nF, Capacitor_SMD:C_0603_1608Metric, F.Cu at (-55.0, 3.25)
- added FB19: 200mA 1kR, Inductor_SMD:L_0805_2012Metric, F.Cu at (-72.6, 19.4)
- added J22: RJ45_Hanrun_HR911105A_Horizontal, Connector_RJ:RJ45_Hanrun_HR911105A_Horizontal, F.Cu at (-99.6, 47.4)
- added R231: 12.1k, Resistor_SMD:R_0603_1608Metric, F.Cu at (-28.4, -1.76)
- added R232: 270R, Resistor_SMD:R_0603_1608Metric, F.Cu at (-109.2, 42.0)
- added R233: 12.1k, Resistor_SMD:R_0603_1608Metric, F.Cu at (-55.0, 8.28)
- added R234: 270R, Resistor_SMD:R_0603_1608Metric, F.Cu at (-109.8, 62.0)
- added RN1: 49.9R, Resistor_SMD:R_Array_Concave_4x0603, F.Cu at (-93.0, 46.8)
- added U27: CD4067BMT/TR, Package_SO:TSSOP-24_4.4x7.8mm_P0.65mm, F.Cu at (-46.6, 24.4)
- added U28: CD4067BMT/TR, Package_SO:TSSOP-24_4.4x7.8mm_P0.65mm, F.Cu at (-37.9, 24.4)
- added U29: CH340C, Package_SO:SOIC-16_3.9x9.9mm_P1.27mm, F.Cu at (-97.4, 69.0)
- added U30: LAN8720A, Package_DFN_QFN:QFN-24-1EP_4x4mm_P0.5mm_EP2.6x2.6mm, F.Cu at (-88.5, 51.3)
- Q11, Q12, Q17, Q18, Q23, Q24, Q29, Q30, Q35, Q36, Q41, Q42, Q47, Q48, Q5, Q53, Q54, Q6: value STN2610D -> HL20N04; footprint Package_TO_SOT_SMD:TO-252-2 -> Package_TO_SOT_SMD:SOT-89-3
- U15: value ESP32-S2-WROVER -> ESP32-WROOM-32; footprint RF_Module:ESP32-S2-WROVER -> RF_Module:ESP32-WROOM-32D
- moved D51 651.9 mm to (741.7, 174.4), turned to -90 degrees
- moved D52 648.7 mm to (739.1, 174.4), turned to -90 degrees
- moved R149 630.1 mm to (716.5, 169.3), turned to -90 degrees
- moved C41 628.5 mm to (706.4, 157.3), turned to -90 degrees
- moved R150 626.9 mm to (713.9, 169.3), turned to -90 degrees
- moved D93 461.9 mm to (580.2, 220.3), turned to -90 degrees
- moved D94 458.5 mm to (577.6, 220.3), turned to -90 degrees
- moved R223 442.5 mm to (554.9, 215.2), turned to -90 degrees
- moved R224 439.1 mm to (552.4, 215.2), turned to -90 degrees
- moved C60 439.1 mm to (544.9, 203.2), turned to -90 degrees
- moved D67 434.8 mm to (447.0, 312.5), turned to -90 degrees
- moved D68 431.2 mm to (444.4, 312.5), turned to -90 degrees
- moved R199 421.2 mm to (421.7, 307.4), turned to -90 degrees
- moved R200 417.7 mm to (419.2, 307.4), turned to -90 degrees
- moved C55 414.6 mm to (411.7, 295.4), turned to -90 degrees
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Connections:
- net /Input multiplexer/D_{In}0 renamed /DC Output channels/D_{In}0
- C24 pad 2: /DC Output channels/A_{In}3 -> /DC Output channels/A_{In}5
- C25 pad 2: /DC Output channels/A_{In}4 -> /DC Output channels/A_{In}6
- C29 pad 2: /DC Output channels/A_{In}1 -> /DC Output channels/A_{In}9
- C30 pad 2: /DC Output channels/A_{In}2 -> /DC Output channels/A_{In}10
- C34 pad 2: /DC Output channels/A_{In}1 -> /DC Output channels/A_{In}11
- C35 pad 2: /DC Output channels/A_{In}2 -> /DC Output channels/A_{In}12
- C39 pad 2: /DC Output channels/A_{In}1 -> /DC Output channels/A_{In}13
- C40 pad 2: /DC Output channels/A_{In}2 -> /DC Output channels/A_{In}14
- C44 pad 2: /DC Output channels/A_{In}1 -> /DC Output channels/A_{In}7
- C45 pad 2: /DC Output channels/A_{In}2 -> /DC Output channels/A_{In}8
- C53 pad 2: /DC Output channels/A_{In}1 -> /DC Output channels/A_{In}15
- C54 pad 2: /DC Output channels/A_{In}2 -> /DC Output channels/A_{In}16
- C58 pad 2: /DC Output channels/A_{In}1 -> /DC Output channels/A_{In}17
- C59 pad 2: /DC Output channels/A_{In}2 -> /DC Output channels/A_{In}18
- D70 pad 2: /DC Output channels/5V output #1/O2+ -> /DC Output channels/5V output #1/O2-
- D72 pad 2: /DC Output channels/5V output #2/O2+ -> /DC Output channels/5V output #2/O2-
- D74 pad 2: /DC Output channels/5V output #3/O2+ -> /DC Output channels/5V output #3/O2-
- D76 pad 2: /DC Output channels/24V output #1/O2+ -> /DC Output channels/24V output #1/O2-
- D78 pad 2: /DC Output channels/12V output #1/O2+ -> /DC Output channels/12V output #1/O2-
- D80 pad 2: /DC Output channels/12V output #2/O2+ -> /DC Output channels/12V output #2/O2-
- D82 pad 2: /DC Output channels/12V output #3/O2+ -> /DC Output channels/12V output #3/O2-
- D84 pad 2: /DC Output channels/9V output #1/O2+ -> /DC Output channels/9V output #1/O2-
- D86 pad 2: /DC Output channels/9V output #2/O2+ -> /DC Output channels/9V output #2/O2-
- J11 pad 2: /DC Output channels/12V output #2/O2+ -> /DC Output channels/12V output #2/O2-
- J13 pad 2: /DC Output channels/12V output #3/O2+ -> /DC Output channels/12V output #3/O2-
- J15 pad 2: /DC Output channels/24V output #1/O2+ -> /DC Output channels/24V output #1/O2-
- J17 pad 2: /DC Output channels/9V output #1/O2+ -> /DC Output channels/9V output #1/O2-
- J19 pad 2: /DC Output channels/9V output #2/O2+ -> /DC Output channels/9V output #2/O2-
- J20 pad A6: /MCU/USB-D+ -> /USB/USB-D+
- J20 pad A7: /MCU/USB-D- -> /USB/USB-D-
- J20 pad B6: /MCU/USB-D+ -> /USB/USB-D+
- J20 pad B7: /MCU/USB-D- -> /USB/USB-D-
- J3 pad 2: /DC Output channels/5V output #1/O2+ -> /DC Output channels/5V output #1/O2-
- J5 pad 2: /DC Output channels/5V output #2/O2+ -> /DC Output channels/5V output #2/O2-
- J7 pad 2: /DC Output channels/5V output #3/O2+ -> /DC Output channels/5V output #3/O2-
- J9 pad 2: /DC Output channels/12V output #1/O2+ -> /DC Output channels/12V output #1/O2-
- R115 pad 1: /DC Output channels/A_{In}1 -> /DC Output channels/A_{In}11
- R116 pad 1: /DC Output channels/A_{In}2 -> /DC Output channels/A_{In}12
- R120 pad 1: /DC Output channels/12V output #2/O2+ -> /DC Output channels/12V output #2/O2-
- R122 pad 2: /DC Output channels/12V output #2/O2+ -> /DC Output channels/12V output #2/O2-
- R139 pad 1: /DC Output channels/A_{In}1 -> /DC Output channels/A_{In}13
- R140 pad 1: /DC Output channels/A_{In}2 -> /DC Output channels/A_{In}14
- R144 pad 1: /DC Output channels/12V output #3/O2+ -> /DC Output channels/12V output #3/O2-
- R146 pad 2: /DC Output channels/12V output #3/O2+ -> /DC Output channels/12V output #3/O2-
- R163 pad 1: /DC Output channels/A_{In}1 -> /DC Output channels/A_{In}7
- R164 pad 1: /DC Output channels/A_{In}2 -> /DC Output channels/A_{In}8
- R168 pad 1: /DC Output channels/24V output #1/O2+ -> /DC Output channels/24V output #1/O2-
- R170 pad 2: /DC Output channels/24V output #1/O2+ -> /DC Output channels/24V output #1/O2-
- R189 pad 1: /DC Output channels/A_{In}1 -> /DC Output channels/A_{In}15
- R190 pad 1: /DC Output channels/A_{In}2 -> /DC Output channels/A_{In}16
- R194 pad 1: /DC Output channels/9V output #1/O2+ -> /DC Output channels/9V output #1/O2-
- R196 pad 2: /DC Output channels/9V output #1/O2+ -> /DC Output channels/9V output #1/O2-
- R213 pad 1: /DC Output channels/A_{In}1 -> /DC Output channels/A_{In}17
- R214 pad 1: /DC Output channels/A_{In}2 -> /DC Output channels/A_{In}18
- R218 pad 1: /DC Output channels/9V output #2/O2+ -> /DC Output channels/9V output #2/O2-
- R220 pad 2: /DC Output channels/9V output #2/O2+ -> /DC Output channels/9V output #2/O2-
- R226 pad 1: +3V3 -> +3.3V
- R229 pad 1: +3V3 -> +3.3V
- R229 pad 2: Net-(U15-IO00) -> ESP32-BOOT
- R230 pad 1: +3V3 -> GND
- R230 pad 2: Net-(U15-IO02) -> Net-(U15-IO2)
- R24 pad 1: /DC Output channels/5V output #1/O2+ -> /DC Output channels/5V output #1/O2-
- R26 pad 2: /DC Output channels/5V output #1/O2+ -> /DC Output channels/5V output #1/O2-
- R48 pad 1: /DC Output channels/5V output #2/O2+ -> /DC Output channels/5V output #2/O2-
- R50 pad 2: /DC Output channels/5V output #2/O2+ -> /DC Output channels/5V output #2/O2-
- R67 pad 1: /DC Output channels/A_{In}3 -> /DC Output channels/A_{In}5
- R68 pad 1: /DC Output channels/A_{In}4 -> /DC Output channels/A_{In}6
- R72 pad 1: /DC Output channels/5V output #3/O2+ -> /DC Output channels/5V output #3/O2-
- R74 pad 2: /DC Output channels/5V output #3/O2+ -> /DC Output channels/5V output #3/O2-
- R91 pad 1: /DC Output channels/A_{In}1 -> /DC Output channels/A_{In}9
- R92 pad 1: /DC Output channels/A_{In}2 -> /DC Output channels/A_{In}10
- R96 pad 1: /DC Output channels/12V output #1/O2+ -> /DC Output channels/12V output #1/O2-
- R98 pad 2: /DC Output channels/12V output #1/O2+ -> /DC Output channels/12V output #1/O2-
- U10 pad 12: /DC Output channels/12V output #1/O2+ -> /DC Output channels/12V output #1/O2-
- U10 pad 14: /DC Output channels/A_{In}2 -> /DC Output channels/A_{In}10
- U10 pad 3: /DC Output channels/A_{In}1 -> /DC Output channels/A_{In}9
- U10 pad 7: /DC Output channels/A_{In}1 -> /DC Output channels/A_{In}9
- U10 pad 9: /DC Output channels/A_{In}2 -> /DC Output channels/A_{In}10
- U11 pad 12: /DC Output channels/12V output #2/O2+ -> /DC Output channels/12V output #2/O2-
- U11 pad 14: /DC Output channels/A_{In}2 -> /DC Output channels/A_{In}12
- U11 pad 3: /DC Output channels/A_{In}1 -> /DC Output channels/A_{In}11
- U11 pad 7: /DC Output channels/A_{In}1 -> /DC Output channels/A_{In}11
- U11 pad 9: /DC Output channels/A_{In}2 -> /DC Output channels/A_{In}12
- U12 pad 12: /DC Output channels/24V output #1/O2+ -> /DC Output channels/24V output #1/O2-
- U12 pad 14: /DC Output channels/A_{In}2 -> /DC Output channels/A_{In}8
- U12 pad 3: /DC Output channels/A_{In}1 -> /DC Output channels/A_{In}7
- U12 pad 7: /DC Output channels/A_{In}1 -> /DC Output channels/A_{In}7
- U12 pad 9: /DC Output channels/A_{In}2 -> /DC Output channels/A_{In}8
- U14 pad 1: /MCU/USB-D+ -> /USB/USB-D+
- U14 pad 3: /MCU/USB-D- -> /USB/USB-D-
- U14 pad 4: /MCU/USB-D- -> /USB/USB-D-
- U14 pad 6: /MCU/USB-D+ -> /USB/USB-D+
- U15 pad 10: unconnected-(U15-IO07-Pad10) -> /MCU/ESP32-RMII-RXD0
- U15 pad 11: unconnected-(U15-IO08-Pad11) -> /MCU/ESP32-RMII-RXD1
- U15 pad 12: unconnected-(U15-IO09-Pad12) -> /MCU/ESP32-RMII-CRSDV
- U15 pad 14: unconnected-(U15-IO11-Pad14) -> /MCU/DO4
- U15 pad 15: unconnected-(U15-IO12-Pad15) -> GND
- U15 pad 2: +3V3 -> +3.3V
- U15 pad 22: /MCU/USB-D- -> unconnected-(U15-SDI/SD1-Pad22)
- U15 pad 23: /MCU/USB-D+ -> unconnected-(U15-IO15-Pad23)
- U15 pad 24: unconnected-(U15-IO21-Pad24) -> Net-(U15-IO2)
- U15 pad 25: unconnected-(U15-IO26-Pad25) -> ESP32-BOOT
- U15 pad 26: GND -> unconnected-(U15-IO4-Pad26)
- U15 pad 28: unconnected-(U15-IO34-Pad28) -> /MCU/ESP32-RMII-REFCLKOUT
- U15 pad 3: Net-(U15-IO00) -> ESP32-~{RST}
- U15 pad 30: unconnected-(U15-IO36-Pad30) -> /MCU/ESP32-RMII-MDIO
- U15 pad 31: unconnected-(U15-IO37-Pad31) -> /MCU/ESP32-RMII-TXD0
- U15 pad 33: unconnected-(U15-IO39-Pad33) -> /MCU/ESP32-RMII-TX-EN
- U15 pad 34: unconnected-(U15-IO40-Pad34) -> ESP32-UART-RX
- U15 pad 35: unconnected-(U15-IO41-Pad35) -> ESP32-UART-TX
- U15 pad 36: unconnected-(U15-IO42-Pad36) -> /MCU/ESP32-RMII-TXD1
- U15 pad 37: unconnected-(U15-TXD0-Pad37) -> /MCU/ESP32-RMII-MDC
- U15 pad 38: unconnected-(U15-RXD0-Pad38) -> GND
- U15 pad 39: unconnected-(U15-IO45-Pad39) -> GND
- U15 pad 4: unconnected-(U15-IO01-Pad4) -> /MCU/DI1
- U15 pad 5: Net-(U15-IO02) -> /MCU/DI2
- U16 pad 11: /Output multiplexer/SCLK -> /Input multiplexer/SCLK
- U16 pad 12: /Output multiplexer/LOAD -> /Input multiplexer/~{LOAD}
- U17 pad 11: /Output multiplexer/SCLK -> /Input multiplexer/SCLK
- U17 pad 12: /Output multiplexer/LOAD -> /Input multiplexer/~{LOAD}
- U18 pad 11: /Output multiplexer/SCLK -> /Input multiplexer/SCLK
- U18 pad 12: /Output multiplexer/LOAD -> /Input multiplexer/~{LOAD}
- U19 pad 11: /Output multiplexer/SCLK -> /Input multiplexer/SCLK
- U19 pad 12: /Output multiplexer/LOAD -> /Input multiplexer/~{LOAD}
- U20 pad 11: /Output multiplexer/SCLK -> /Input multiplexer/SCLK
- U20 pad 12: /Output multiplexer/LOAD -> /Input multiplexer/~{LOAD}
- U21 pad 11: /Output multiplexer/SCLK -> /Input multiplexer/SCLK
- U21 pad 12: /Output multiplexer/LOAD -> /Input multiplexer/~{LOAD}
- U22 pad 11: /Output multiplexer/SCLK -> /Input multiplexer/SCLK
- U22 pad 12: /Output multiplexer/LOAD -> /Input multiplexer/~{LOAD}
- U23 pad 12: /Input multiplexer/D_{In}1 -> /DC Output channels/D_{In}1
- U23 pad 13: /Input multiplexer/D_{In}2 -> /DC Output channels/D_{In}2
- U23 pad 14: /Input multiplexer/D_{In}3 -> /DC Output channels/D_{In}3
- U23 pad 3: /Input multiplexer/D_{In}4 -> /DC Output channels/D_{In}4
- U23 pad 4: /Input multiplexer/D_{In}5 -> /DC Output channels/D_{In}5
- U23 pad 5: /Input multiplexer/D_{In}6 -> /DC Output channels/D_{In}6
- U23 pad 6: /Input multiplexer/D_{In}7 -> /DC Output channels/D_{In}7
- U24 pad 11: /Input multiplexer/D_{In}8 -> /DC Output channels/D_{In}8
- U24 pad 12: /Input multiplexer/D_{In}9 -> /DC Output channels/D_{In}9
- U24 pad 13: /Input multiplexer/D_{In}10 -> /DC Output channels/D_{In}10
- U24 pad 14: /Input multiplexer/D_{In}11 -> /DC Output channels/D_{In}11
- U24 pad 3: /Input multiplexer/D_{In}12 -> /DC Output channels/D_{In}12
- U24 pad 4: /Input multiplexer/D_{In}13 -> /DC Output channels/D_{In}13
- U24 pad 5: /Input multiplexer/D_{In}14 -> /DC Output channels/D_{In}14
- U24 pad 6: /Input multiplexer/D_{In}15 -> /DC Output channels/D_{In}15
- U25 pad 11: /Input multiplexer/D_{In}8 -> /DC Output channels/D_{In}8
- U25 pad 12: /Input multiplexer/D_{In}9 -> /DC Output channels/D_{In}9
- U25 pad 13: /Input multiplexer/D_{In}10 -> /DC Output channels/D_{In}10
- U25 pad 14: /Input multiplexer/D_{In}11 -> /DC Output channels/D_{In}11
- U25 pad 3: /Input multiplexer/D_{In}12 -> /DC Output channels/D_{In}12
- U25 pad 4: /Input multiplexer/D_{In}13 -> /DC Output channels/D_{In}13
- U25 pad 5: /Input multiplexer/D_{In}14 -> /DC Output channels/D_{In}14
- U25 pad 6: /Input multiplexer/D_{In}15 -> /DC Output channels/D_{In}15
- U26 pad 11: /Input multiplexer/D_{In}16 -> /DC Output channels/D_{In}16
- U26 pad 12: /Input multiplexer/D_{In}17 -> /DC Output channels/D_{In}17
- U26 pad 13: /Input multiplexer/D_{In}18 -> /DC Output channels/D_{In}18
- U4 pad 12: /DC Output channels/5V output #1/O2+ -> /DC Output channels/5V output #1/O2-
- U5 pad 12: /DC Output channels/12V output #3/O2+ -> /DC Output channels/12V output #3/O2-
- U5 pad 14: /DC Output channels/A_{In}2 -> /DC Output channels/A_{In}14
- U5 pad 3: /DC Output channels/A_{In}1 -> /DC Output channels/A_{In}13
- U5 pad 7: /DC Output channels/A_{In}1 -> /DC Output channels/A_{In}13
- U5 pad 9: /DC Output channels/A_{In}2 -> /DC Output channels/A_{In}14
- U6 pad 12: /DC Output channels/9V output #1/O2+ -> /DC Output channels/9V output #1/O2-
- U6 pad 14: /DC Output channels/A_{In}2 -> /DC Output channels/A_{In}16
- U6 pad 3: /DC Output channels/A_{In}1 -> /DC Output channels/A_{In}15
- U6 pad 7: /DC Output channels/A_{In}1 -> /DC Output channels/A_{In}15
- U6 pad 9: /DC Output channels/A_{In}2 -> /DC Output channels/A_{In}16
- U7 pad 12: /DC Output channels/9V output #2/O2+ -> /DC Output channels/9V output #2/O2-
- U7 pad 14: /DC Output channels/A_{In}2 -> /DC Output channels/A_{In}18
- U7 pad 3: /DC Output channels/A_{In}1 -> /DC Output channels/A_{In}17
- U7 pad 7: /DC Output channels/A_{In}1 -> /DC Output channels/A_{In}17
- U7 pad 9: /DC Output channels/A_{In}2 -> /DC Output channels/A_{In}18
- U8 pad 12: /DC Output channels/5V output #2/O2+ -> /DC Output channels/5V output #2/O2-
- U9 pad 12: /DC Output channels/5V output #3/O2+ -> /DC Output channels/5V output #3/O2-
- U9 pad 14: /DC Output channels/A_{In}4 -> /DC Output channels/A_{In}6
- U9 pad 3: /DC Output channels/A_{In}3 -> /DC Output channels/A_{In}5
- U9 pad 7: /DC Output channels/A_{In}3 -> /DC Output channels/A_{In}5
- U9 pad 9: /DC Output channels/A_{In}4 -> /DC Output channels/A_{In}6
Routing:
- net GND: track 0.00 -> 42.9 mm, vias 0 -> 3
- net /USB/USB-D+: track 0.00 -> 15.9 mm, vias 0 -> 2
- net VUSB: track 0.00 -> 15.5 mm, vias 0 -> 2
- net /MCU/Ethernet/PHY-RXP: track 0.00 -> 14.0 mm
- net /USB/USB-D-: track 0.00 -> 13.0 mm
- net /MCU/Ethernet/PHY-RXN: track 0.00 -> 13.0 mm
- net /MCU/Ethernet/PHY-TXN: track 0.00 -> 11.8 mm
- net /MCU/Ethernet/PHY-TXP: track 0.00 -> 11.2 mm
- net +3.3V: track 0.00 -> 11.0 mm
- net Net-(J22-Pad11): track 0.00 -> 7.00 mm
- net Net-(U7B--): track 0.00 -> 6.35 mm
- net Net-(U5B--): track 0.00 -> 6.35 mm
- net Net-(U10B--): track 0.00 -> 6.35 mm
- net Net-(U4B--): track 0.00 -> 6.35 mm
- net Net-(U9B--): track 0.00 -> 6.35 mm
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