File: OpenPowerDistributor/OpenPowerDistribution.kicad_sch (KiCad schematic)
At the start: 0 parts

Commit message: Analog multiplexer work
Other:
- added sheet Analog multiplexer (Analog multiplexer.kicad_sch)
- sheet Input multiplexer ports: added D_{In}, MUX-Load, SPI-MISO, SPI-SCLK, SPI-~{CS}; removed none
- sheet MCU ports: added AIN1, AIN2; removed none
- note removed: "30V power supply for high-side FET gate power"
Changed lines of the file:
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@@
 (kicad_sch (version 20230121) (generator eeschema)
   (paper "A4")
-  (bus (pts (xy 226.06 46.99) (xy 236.22 46.99))
-    (stroke (width 0) (type default))
-  )
-  (text "30V power supply for high-side FET gate power" (at 54.61 24.13 0)
-    (effects (font (size 3 3)) (justify left bottom))
+  (junction (at 229.87 46.99) (diameter 0) (color 0 0 0 0)
+  )
+  (bus (pts (xy 229.87 68.58) (xy 229.87 46.99))
+    (stroke (width 0) (type default))
+  )
+  (wire (pts (xy 186.69 76.2) (xy 193.04 76.2))
+    (stroke (width 0) (type default))
+  )
+  (wire (pts (xy 193.04 71.12) (xy 189.23 71.12))
+    (stroke (width 0) (type default))
+  )
+  (bus (pts (xy 229.87 46.99) (xy 236.22 46.99))
+    (stroke (width 0) (type default))
+  )
+  (wire (pts (xy 189.23 71.12) (xy 189.23 46.99))
+    (stroke (width 0) (type default))
+  )
+  (wire (pts (xy 193.04 54.61) (xy 186.69 54.61))
+    (stroke (width 0) (type default))
+  )
+  (wire (pts (xy 189.23 46.99) (xy 193.04 46.99))
+    (stroke (width 0) (type default))
+  )
+  (wire (pts (xy 186.69 54.61) (xy 186.69 76.2))
+    (stroke (width 0) (type default))
+  )
+  (bus (pts (xy 226.06 46.99) (xy 229.87 46.99))
+    (stroke (width 0) (type default))
+  )
+  (bus (pts (xy 226.06 68.58) (xy 229.87 68.58))
+    (stroke (width 0) (type default))
   )
   (sheet (at 236.22 44.45) (size 17.78 8.89) (fields_autoplaced)
@@
     )
   )
-  (sheet (at 128.27 53.34) (size 43.18 33.02) (fields_autoplaced)
-    (stroke (width 0.1524) (type solid))
-    (fill (color 0 0 0 0.0000))
-    (property "Sheetname" "MCU" (at 128.27 52.6284 0)
-      (effects (font (size 1.27 1.27)) (justify left bottom))
-    )
-    (property "Sheetfile" "MCU.kicad_sch" (at 128.27 86.9446 0)
-      (effects (font (size 1.27 1.27)) (justify left top))
+  (sheet (at 193.04 86.36) (size 31.75 13.97) (fields_autoplaced)
+    (stroke (width 0.1524) (type solid))
+    (fill (color 0 0 0 0.0000))
+    (property "Sheetname" "Analog multiplexer" (at 193.04 85.6484 0)
+      (effects (font (size 1.27 1.27)) (justify left bottom))
+    )
+    (property "Sheetfile" "Analog multiplexer.kicad_sch" (at 193.04 100.9146 0)
+      (effects (font (size 1.27 1.27)) (justify left top))
+    )
+    (pin "AIN2" input (at 193.04 96.52 180)
+      (effects (font (size 1.27 1.27)) (justify left))
+    )
+    (pin "AIN1" input (at 193.04 93.98 180)
+      (effects (font (size 1.27 1.27)) (justify left))
+    )
+    (pin "AMUX" input (at 193.04 90.17 180)
+      (effects (font (size 1.27 1.27)) (justify left))
+    )
+    (instances
+      (project "OpenPowerDistribution"
+        (path "/df87b081-37a2-452c-8581-7eff2c408a17" (page "21"))
+      )
+    )
+  )
+  (sheet (at 124.46 41.91) (size 40.64 16.51) (fields_autoplaced)
+    (stroke (width 0.1524) (type solid))
+    (fill (color 0 0 0 0.0000))
+    (property "Sheetname" "MCU" (at 124.46 41.1984 0)
+      (effects (font (size 1.27 1.27)) (justify left bottom))
+    )
+    (property "Sheetfile" "MCU.kicad_sch" (at 124.46 59.0046 0)
+      (effects (font (size 1.27 1.27)) (justify left top))
+    )
+    (pin "AIN1" input (at 165.1 45.72 0)
+      (effects (font (size 1.27 1.27)) (justify right))
+    )
+    (pin "AIN2" input (at 165.1 48.26 0)
+      (effects (font (size 1.27 1.27)) (justify right))
     )
     (instances
@@
       (effects (font (size 1.27 1.27)) (justify left top))
     )
-    (instances
+    (pin "D_{In}" output (at 226.06 68.58 0)
+      (effects (font (size 1.27 1.27)) (justify right))
+    )
+    (pin "SPI-MISO" output (at 193.04 68.58 180)
+      (effects (font (size 1.27 1.27)) (justify left))
+    )
+    (pin "MUX-Load" input (at 193.04 76.2 180)
+      (effects (font (size 1.27 1.27)) (justify left))
+    )
+    (pin "SPI-SCLK" input (at 193.04 71.12 180)
+      (effects (font (size 1.27 1.27)) (justify left))
+    )
+    (pin "SPI-~{CS}" input (at 193.04 73.66 180)
+      (effects (font (size 1.27 1.27)) (justify left))
+    )
+    (instances

Commit message: Work mostly on Ethernet schematic
Other:
- added sheet USB (USB.kicad_sch)
- sheet Analog multiplexer ports: added AMUX-Out; removed AIN1, AIN2
Changed lines of the file:
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@@
     )
   )
-  (sheet (at 193.04 86.36) (size 31.75 13.97) (fields_autoplaced)
+  (sheet (at 193.04 86.36) (size 31.75 7.62) (fields_autoplaced)
     (stroke (width 0.1524) (type solid))
     (fill (color 0 0 0 0.0000))
@@
       (effects (font (size 1.27 1.27)) (justify left bottom))
     )
-    (property "Sheetfile" "Analog multiplexer.kicad_sch" (at 193.04 100.9146 0)
+    (property "Sheetfile" "Analog multiplexer.kicad_sch" (at 193.04 94.5646 0)
       (effects (font (size 1.27 1.27)) (justify left top))
     )
-    (pin "AIN2" input (at 193.04 96.52 180)
-      (effects (font (size 1.27 1.27)) (justify left))
+    (pin "AMUX" input (at 224.79 90.17 0)
+      (effects (font (size 1.27 1.27)) (justify right))
     )
-    (pin "AIN1" input (at 193.04 93.98 180)
-      (effects (font (size 1.27 1.27)) (justify left))
-    )
-    (pin "AMUX" input (at 193.04 90.17 180)
+    (pin "AMUX-Out" output (at 193.04 90.17 180)
       (effects (font (size 1.27 1.27)) (justify left))
     )
@@
       )
     )
+  )
+  (sheet (at 124.46 68.58) (size 38.1 15.24) (fields_autoplaced)
+    (stroke (width 0.1524) (type solid))
+    (fill (color 0 0 0 0.0000))
+    (property "Sheetname" "USB" (at 124.46 67.8684 0)
+      (effects (font (size 1.27 1.27)) (justify left bottom))
+    )
+    (property "Sheetfile" "USB.kicad_sch" (at 124.46 84.4046 0)
+      (effects (font (size 1.27 1.27)) (justify left top))
+    )
+    (instances
+      (project "OpenPowerDistribution"
+        (path "/df87b081-37a2-452c-8581-7eff2c408a17" (page "23"))
+      )
+    )
